File: cad/stoerbert.kicad_pcb (KiCad board)
At the start: 2 copper layers, 32 parts, among them SW1 OmronB3F, SW2 OmronB3F, SW3 OmronB3F, SW4 OmronB3F, SW5 OmronB3F, SW6 OmronB3F, SW7 OmronB3F, SW8 OmronB3F, SW9 OmronB3F, U1 4021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

Commit message: Updated PCB
Parts:
- J_POT1: footprint Connector_PinHeader_2.00mm:PinHeader_1x03_P2.00mm_Vertical -> cad:PinHeader_1x03_P2.00mm_Vertical_large
- U1, U2: footprint Package_DIP:DIP-16_W7.62mm -> cad:DIP-16_W7.62mm_large; moved to B.Cu
- moved R1 22.1 mm to (-193.2, -901.0)
- moved R9 19.8 mm to (-161.3, -900.5)
- moved R15 17.0 mm to (-138.3, -885.0)
- moved U2 16.2 mm to (-153.2, -883.5)
- moved R8 16.1 mm to (-193.2, -887.0)
- moved J_POT1 15.7 mm to (-127.2, -904.5)
- moved U1 15.6 mm to (-186.2, -883.5)
- moved R16 15.0 mm to (-161.2, -886.5)
- moved R7 14.7 mm to (-170.7, -886.5)
- moved R2 12.6 mm to (-193.3, -897.5)
- moved R10 11.6 mm to (-161.3, -897.0)
- moved J_DATA1 11.6 mm to (-131.2, -893.5), turned to 180 degrees
- moved R14 9.42 mm to (-138.3, -888.5)
- moved R12 7.05 mm to (-161.3, -890.0)
- moved R4 6.72 mm to (-193.3, -890.5)
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Connections:
- J_DATA1 pad 1: +5V -> Net-(J_DATA1-Pad1)
- J_DATA1 pad 2: GND -> Net-(J_DATA1-Pad2)
- J_DATA1 pad 4: Net-(J_DATA1-Pad4) -> GND
- J_DATA1 pad 5: Net-(J_DATA1-Pad5) -> +5V
- SW1 pad 3: Net-(R2-Pad2) -> Net-(R4-Pad2)
- SW5 pad 3: Net-(R7-Pad2) -> Net-(R5-Pad2)
- SW6 pad 3: Net-(R10-Pad2) -> Net-(R12-Pad2)
- SW7 pad 3: Net-(R4-Pad2) -> Net-(R2-Pad2)
- SW8 pad 3: Net-(R12-Pad2) -> Net-(R10-Pad2)
- SW_NEXT1 pad 3: Net-(R15-Pad2) -> Net-(R13-Pad2)
- SW_PLAY1 pad 3: Net-(R16-Pad2) -> Net-(R9-Pad2)
- SW_PREV1 pad 3: Net-(R8-Pad2) -> Net-(R1-Pad2)
- U1 pad 10: Net-(J_DATA1-Pad4) -> Net-(J_DATA1-Pad2)
- U1 pad 3: Net-(J_DATA1-Pad3) -> Net-(J_DATA1-Pad1)
- U1 pad 9: Net-(J_DATA1-Pad5) -> Net-(J_DATA1-Pad3)
- U2 pad 10: Net-(J_DATA1-Pad4) -> Net-(J_DATA1-Pad2)
- U2 pad 9: Net-(J_DATA1-Pad5) -> Net-(J_DATA1-Pad3)
Routing:
- net Net-(R5-Pad2): track 6.54 -> 106.7 mm
- net Net-(R7-Pad2): track 91.1 -> 7.48 mm
- net Net-(J_DATA1-Pad1): track 0.00 -> 75.8 mm
- net Net-(J_DATA1-Pad4): track 75.5 -> 0.00 mm, vias 2 -> 0
- net Net-(J_DATA1-Pad5): track 73.8 -> 0.00 mm, vias 2 -> 0
- net Net-(J_DATA1-Pad2): track 0.00 -> 70.2 mm, vias 0 -> 2
- net Net-(R2-Pad2): track 135.5 -> 75.1 mm
- net Net-(R4-Pad2): track 76.6 -> 131.9 mm
- net Net-(J_DATA1-Pad3): track 115.0 -> 65.6 mm, vias 3 -> 2
- net GND: track 212.2 -> 261.3 mm, vias 4 -> 6
- net Net-(R13-Pad2): track 5.54 -> 52.6 mm
- net Net-(R10-Pad2): track 110.8 -> 71.7 mm
- net +5V: track 412.3 -> 447.0 mm, vias 4 -> 6
- net Net-(R15-Pad2): track 37.8 -> 6.76 mm
- net Net-(R12-Pad2): track 75.4 -> 106.3 mm
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Other:
- board text added: "Stoerbert rev1.1 for Luka"
