File: cad/stoerbert.sch (KiCad schematic (older format))
At the start: 32 parts, among them SW1 OmronB3F, SW2 OmronB3F, SW3 OmronB3F, SW4 OmronB3F, SW5 OmronB3F, SW6 OmronB3F, SW7 OmronB3F, SW8 OmronB3F, SW9 OmronB3F, U1 4021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

Commit message: Updated PCB
Parts:
- U1, U2: footprint Package_DIP:DIP-16_W7.62mm -> cad:DIP-16_W7.62mm_large
Connections:
- net +5V: now also J_DATA1.5 (Pin_5); no longer J_DATA1.1 (Pin_1)
- net GND: now also J_DATA1.4 (Pin_4); no longer J_DATA1.2 (Pin_2)
- net at R2.2, U1.6 (D1): now also SW7.3; no longer SW1.3
- net at R7.2, U1.15 (D6): no longer SW5.3
- net at R10.2, U2.6 (D1): now also SW8.3; no longer SW6.3
- net at R4.2, U1.4 (D3): now also SW1.3; no longer SW7.3
- net at R12.2, U2.4 (D3): now also SW6.3; no longer SW8.3
- net at R8.2, U1.1 (D7): no longer SW_PREV1.3
- net at R16.2, U2.1 (D7): no longer SW_PLAY1.3
- net at R15.2, U2.15 (D6): no longer SW_NEXT1.3
- net at R13.2, U2.13 (D4): now also SW_NEXT1.3
- net at R9.2, U2.7 (D0): now also SW_PLAY1.3
- net at R5.2, U1.13 (D4): now also SW5.3
- net at R1.2, U1.7 (D0): now also SW_PREV1.3
- net at U1.10 (CP), U2.10 (CP): now also J_DATA1.2 (Pin_2); no longer J_DATA1.4 (Pin_4)
- net at U1.9 (PL), U2.9 (PL): now also J_DATA1.3 (Pin_3); no longer J_DATA1.5 (Pin_5)
- net at U1.3 (Q7): now also J_DATA1.1 (Pin_1); no longer J_DATA1.3 (Pin_3)
